File: UNOvx.sch (KiCad schematic (older format))
At the start: 38 parts, among them IC1 BTS462T, J1 Barrel_Jack_Switch, J2 Ext. Power, J3 Conn_01x02_Male, J4 Conn_02x03_Odd_Even, P1 Analog, P2 Power, P3 Digital, P4 Digital, P5 CONN_01X01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

Commit message: Route the switch
Parts:
- IC1: footprint TO-252-5PIN -> kicad-lib:TO-252-5PIN
Changed lines of the file:
@@
 F 0 "IC1" H 7400 9765 50  0000 C CNN
 F 1 "BTS462T" H 7400 9674 50  0000 C CNN
-F 2 "TO-252-5PIN" H 7850 9600 50  0001 L CNN
+F 2 "kicad-lib:TO-252-5PIN" H 7850 9600 50  0001 L CNN
 F 3 "" H 7850 9500 50  0001 L CNN
 F 4 "Smart High-Side Power Switch TO252-5 Infineon BTS462T Intelligent Power Switch, High Side, 4.4A, -10  16V, 5-Pin, TO-252" H 7850 9400 50  0001 L CNN "Description"

Commit message: Fix symbol legs. Add oscillator
Parts:
- removed P5, P6, P7, P8: CONN_01X01, Socket_Arduino_Uno:Arduino_1pin, symbol Connector_Generic:Conn_01x01
- added Y2: 16MHz, Crystal:Resonator_SMD_muRata_CDSCB-2Pin_4.5x2.0mm, symbol Device:Crystal
Connections:
- wire segments 102 -> 108
- no-connect marks 6 -> 1
Other:
- note removed: "Holes"
- moved on the sheet: C3, C5
Changed lines of the file:
@@
 Comment4 ""
 $EndDescr
-NoConn ~ 14650 7000
-Text Notes 15700 1000 0    60   ~ 0
-Holes
 Text Notes 13400 750  0    60   ~ 0
 Shield for Arduino that uses\nthe same pin disposition\nlike "Uno" board Rev 3.
@@
 	1    0    0    -1
 $EndComp
-$Comp
-L Connector_Generic:Conn_01x01 P5
-U 1 1 56D71177
-P 15650 650
-F 0 "P5" V 15750 650 50  0000 C CNN
-F 1 "CONN_01X01" V 15750 650 50  0001 C CNN
-F 2 "Socket_Arduino_Uno:Arduino_1pin" H 15571 724 20  0000 C CNN
-F 3 "" H 15650 650 50  0000 C CNN
-	1    15650 650
-	0    -1   -1   0
-$EndComp
-$Comp
-L Connector_Generic:Conn_01x01 P6
-U 1 1 56D71274
-P 15750 650
-F 0 "P6" V 15850 650 50  0000 C CNN
-F 1 "CONN_01X01" V 15850 650 50  0001 C CNN
-F 2 "Socket_Arduino_Uno:Arduino_1pin" H 15750 650 20  0001 C CNN
-F 3 "" H 15750 650 50  0000 C CNN
-	1    15750 650
-	0    -1   -1   0
-$EndComp
-$Comp
-L Connector_Generic:Conn_01x01 P7
-U 1 1 56D712A8
-P 15850 650
-F 0 "P7" V 15950 650 50  0000 C CNN
-F 1 "CONN_01X01" V 15950 650 50  0001 C CNN
-F 2 "Socket_Arduino_Uno:Arduino_1pin" V 15850 650 20  0001 C CNN
-F 3 "" H 15850 650 50  0000 C CNN
-	1    15850 650
-	0    -1   -1   0
-$EndComp
-$Comp
-L Connector_Generic:Conn_01x01 P8
-U 1 1 56D712DB
-P 15950 650
-F 0 "P8" V 16050 650 50  0000 C CNN
-F 1 "CONN_01X01" V 16050 650 50  0001 C CNN
-F 2 "Socket_Arduino_Uno:Arduino_1pin" H 15874 572 20  0000 C CNN
-F 3 "" H 15950 650 50  0000 C CNN
-	1    15950 650
-	0    -1   -1   0
-$EndComp
-NoConn ~ 15650 850
-NoConn ~ 15750 850
-NoConn ~ 15850 850
-NoConn ~ 15950 850
 Wire Notes Line
 	13375 825  14775 825
@@
 Text Notes 14950 7000 0    60   ~ 0
 1
-Wire Notes Line
-	16050 1000 15550 1000
-Wire Notes Line
-	15550 1000 15550 500
 $Comp
 L MCU_Microchip_ATmega:ATmega328P-PU U1
@@
 L Device:C C5
 U 1 1 5DAC0ECB
-P 3950 9150
-F 0 "C5" H 3835 9104 50  0000 R CNN
-F 1 "22pF" H 3835 9195 50  0000 R CNN
-F 2 "Capacitor_SMD:C_0805_2012Metric" H 3988 9000 50  0001 C CNN
-F 3 "~" H 3950 9150 50  0001 C CNN
-	1    3950 9150
+P 3950 9650
+F 0 "C5" H 3835 9604 50  0000 R CNN
+F 1 "22pF" H 3835 9695 50  0000 R CNN
+F 2 "Capacitor_SMD:C_0805_2012Metric" H 3988 9500 50  0001 C CNN
+F 3 "~" H 3950 9650 50  0001 C CNN
+	1    3950 9650
 	-1   0    0    1
 $EndComp
@@
 L Device:C C3
 U 1 1 5DAC2CA7
-P 2950 9150
-F 0 "C3" H 2835 9104 50  0000 R CNN
-F 1 "22pF" H 2835 9195 50  0000 R CNN
-F 2 "Capacitor_SMD:C_0805_2012Metric" H 2988 9000 50  0001 C CNN
-F 3 "~" H 2950 9150 50  0001 C CNN
-	1    2950 9150
+P 2950 9650
+F 0 "C3" H 2835 9604 50  0000 R CNN
+F 1 "22pF" H 2835 9695 50  0000 R CNN
+F 2 "Capacitor_SMD:C_0805_2012Metric" H 2988 9500 50  0001 C CNN
+F 3 "~" H 2950 9650 50  0001 C CNN
+	1    2950 9650
 	-1   0    0    1
 $EndComp
@@
 L power:GND #PWR04
 U 1 1 5DAC4F01
-P 2950 9300
-F 0 "#PWR04" H 2950 9050 50  0001 C CNN
-F 1 "GND" H 2955 9127 50  0000 C CNN
-F 2 "" H 2950 9300 50  0001 C CNN
-F 3 "" H 2950 9300 50  0001 C CNN
-	1    2950 9300
+P 2950 9800
+F 0 "#PWR04" H 2950 9550 50  0001 C CNN
+F 1 "GND" H 2955 9627 50  0000 C CNN
+F 2 "" H 2950 9800 50  0001 C CNN
+F 3 "" H 2950 9800 50  0001 C CNN
+	1    2950 9800
 	1    0    0    -1
 $EndComp
@@
 L power:GND #PWR09
 U 1 1 5DAC5484
-P 3950 9300
-F 0 "#PWR09" H 3950 9050 50  0001 C CNN
-F 1 "GND" H 3955 9127 50  0000 C CNN
-F 2 "" H 3950 9300 50  0001 C CNN
-F 3 "" H 3950 9300 50  0001 C CNN
-	1    3950 9300
+P 3950 9800
+F 0 "#PWR09" H 3950 9550 50  0001 C CNN
+F 1 "GND" H 3955 9627 50  0000 C CNN
+F 2 "" H 3950 9800 50  0001 C CNN
+F 3 "" H 3950 9800 50  0001 C CNN
+	1    3950 9800
 	1    0    0    -1
 $EndComp
@@
 Connection ~ 2950 8950
 Wire Wire Line
-	2950 8950 2950 9000
-Wire Wire Line
 	3600 8950 3950 8950
 Connection ~ 3950 8950
-Wire Wire Line
-	3950 8950 3950 9000
 $Comp
 L Device:R R7
@@
 $EndComp
 Wire Wire Line
-	14400 6750 14400 7300
+	14400 6750 14400 7000
 $Comp
 L Connector_Generic:Conn_01x06 P1
@@
 $EndComp
 Connection ~ 6800 9700
+$Comp
+L Device:Crystal Y2
+U 1 1 5E07A052
+P 3450 9400
+F 0 "Y2" H 3450 9668 50  0000 C CNN
+F 1 "16MHz" H 3450 9577 50  0000 C CNN
+F 2 "Crystal:Resonator_SMD_muRata_CDSCB-2Pin_4.5x2.0mm" H 3450 9400 50  0001 C CNN
+F 3 "~" H 3450 9400 50  0001 C CNN
+	1    3450 9400
+	1    0    0    -1
+$EndComp
+Wire Wire Line
+	2950 8950 2950 9400
+Wire Wire Line
+	3300 9400 2950 9400
+Connection ~ 2950 9400
+Wire Wire Line
+	2950 9400 2950 9500
+Wire Wire Line
+	3950 8950 3950 9400
+Wire Wire Line
+	3600 9400 3950 9400
+Connection ~ 3950 9400
+Wire Wire Line
+	3950 9400 3950 9500
+Wire Wire Line
+	14650 7000 14400 7000
+Connection ~ 14400 7000
+Wire Wire Line
+	14400 7000 14400 7300
 $EndSCHEMATC

Commit message: No power connector
Parts:
- removed J2: Ext. Power, Connector_PinHeader_2.54mm:PinHeader_1x02_P2.54mm_Vertical, symbol Connector:Conn_01x02_Male
Connections:
- wire segments 108 -> 106
Changed lines of the file:
@@
 	2000 2000 2000 1400
 Connection ~ 2000 2000
-Wire Wire Line
-	2250 1900 2250 1200
 Connection ~ 2250 1200
 NoConn ~ 8000 9500
@@
 Wire Wire Line
 	3600 4400 3600 4000
-Wire Wire Line
-	2000 2000 2250 2000
 Wire Wire Line
 	3500 4400 3500 4000
@@
 $EndComp
 $Comp
-L Connector:Conn_01x02_Male J2
-U 1 1 5DC0B3E2
-P 2450 1900
-F 0 "J2" H 2422 1874 50  0000 R CNN
-F 1 "Ext. Power" H 2422 1783 50  0000 R CNN
-F 2 "Connector_PinHeader_2.54mm:PinHeader_1x02_P2.54mm_Vertical" H 2450 1900 50  0001 C CNN
-F 3 "~" H 2450 1900 50  0001 C CNN
-	1    2450 1900
-	-1   0    0    -1
-$EndComp
-$Comp

Commit message: Layout in 2 layers
No diodes for Rx,Tx
Parts:
- removed D2, D3: Yellow, LED_SMD:LED_0805_2012Metric, symbol Device:LED_ALT
- removed P3: Digital, Socket_Arduino_Uno:Socket_Strip_Arduino_1x10, symbol Connector_Generic:Conn_01x10
- removed R3, R4: 1k, Resistor_SMD:R_0805_2012Metric, symbol Device:R
- added J2: I2C/TWI, Connector_PinHeader_2.54mm:PinHeader_1x02_P2.54mm_Vertical, symbol Connector_Generic:Conn_01x02
- added P3: Digital PB, Socket_Arduino_Uno:Socket_Strip_Arduino_1x06, symbol Connector_Generic:Conn_01x06
- P1: value Analog -> Analog PC
- P2: footprint Socket_Arduino_Uno:Socket_Strip_Arduino_1x08 -> Connector_PinHeader_2.54mm:PinHeader_1x09_P2.54mm_Vertical; symbol Connector_Generic:Conn_01x08 -> Connector_Generic:Conn_01x09
- P4: value Digital -> Digital PD
- U1: symbol MCU_Microchip_ATmega:ATmega328P-PU -> UNOvx-rescue:ATmega328P-PU-MCU_Microchip_ATmega
Connections:
- net labels removed: 10(**/SS), 11(**/MOSI), 12(MISO), 13(SCK), 8, 9(**)
- wire segments 106 -> 98
Other:
- moved on the sheet: D6, J4, R7

Commit message: Update packages to 0805
Parts:
- R2, R5: footprint Capacitor_SMD:C_1210_3225Metric -> Resistor_SMD:R_0805_2012Metric
- R7: footprint Resistor_SMD:R_1210_3225Metric -> Resistor_SMD:R_0805_2012Metric
- U1: symbol UNOvx-rescue:ATmega328P-PU-MCU_Microchip_ATmega -> MCU_Microchip_ATmega:ATmega328P-PU
Changed lines of the file:
@@
 1
 $Comp
-L UNOvx-rescue:ATmega328P-PU-MCU_Microchip_ATmega U1
+L MCU_Microchip_ATmega:ATmega328P-PU U1
 U 1 1 5DA59660
 P 3500 5900
@@
 F 0 "R7" H 12820 6996 50  0000 L CNN
 F 1 "10k" H 12820 6905 50  0000 L CNN
-F 2 "Resistor_SMD:R_1210_3225Metric" V 12680 6950 50  0001 C CNN
+F 2 "Resistor_SMD:R_0805_2012Metric" V 12680 6950 50  0001 C CNN
 F 3 "~" H 12750 6950 50  0001 C CNN
 	1    12750 6950
@@
 F 0 "R2" H 5970 1546 50  0000 L CNN
 F 1 "1k" H 5970 1455 50  0000 L CNN
-F 2 "Capacitor_SMD:C_1210_3225Metric" V 5830 1500 50  0001 C CNN
+F 2 "Resistor_SMD:R_0805_2012Metric" V 5830 1500 50  0001 C CNN
 F 3 "~" H 5900 1500 50  0001 C CNN
 	1    5900 1500
@@
 F 0 "R5" H 6220 1546 50  0000 L CNN
 F 1 "1k" H 6220 1455 50  0000 L CNN
-F 2 "Capacitor_SMD:C_1210_3225Metric" V 6080 1500 50  0001 C CNN
+F 2 "Resistor_SMD:R_0805_2012Metric" V 6080 1500 50  0001 C CNN
 F 3 "~" H 6150 1500 50  0001 C CNN
 	1    6150 1500

Commit message: Rev. B
Parts:
- removed IC1: BTS462T, kicad-lib:TO-252-5PIN, symbol SamacSys_Parts:BTS462T
- removed J3: Conn_01x02_Male, kicad-lib:MKDSN-2.5-1734656, symbol Connector:Conn_01x02_Male
- removed R1: 1M, Resistor_SMD:R_0805_2012Metric, symbol Device:R
- removed Y1: 16MHz, kicad-lib:CR23-crystal-11.3x4.5mm, symbol Device:Crystal
- removed Y2: 16MHz, Crystal:Resonator_SMD_muRata_CDSCB-2Pin_4.5x2.0mm, symbol Device:Crystal
- added D2: YellowTx, LED_SMD:LED_0805_2012Metric_Pad1.15x1.40mm_HandSolder, symbol Device:LED_ALT
- added D3: YellowRx, LED_SMD:LED_0805_2012Metric_Pad1.15x1.40mm_HandSolder, symbol Device:LED_ALT
- added D6: Yellow, LED_SMD:LED_0805_2012Metric_Pad1.15x1.40mm_HandSolder, symbol Device:LED_ALT
- added J2: Conn_01x02, kicad-lib:MKDSN-2.5-1734656, symbol Connector_Generic:Conn_01x02
- added P3: Digital PB, Connector_PinHeader_2.54mm:PinHeader_1x06_P2.54mm_Vertical, symbol Connector_Generic:Conn_01x06
- added P5: Analog PC, Connector_PinHeader_2.54mm:PinHeader_1x06_P2.54mm_Vertical, symbol Connector_Generic:Conn_01x06
- added P7: Digital PD, Connector_PinHeader_2.54mm:PinHeader_1x08_P2.54mm_Vertical, symbol Connector_Generic:Conn_01x08
- added R2, R3: 1k, Resistor_SMD:R_0805_2012Metric_Pad1.15x1.40mm_HandSolder, symbol Device:R
- added R7: 330, Resistor_SMD:R_0805_2012Metric_Pad1.15x1.40mm_HandSolder, symbol Device:R
- added unit 2 of U3
- added Y1: 16MHz, Crystal:Crystal_SMD_Abracon_ABM8G-4Pin_3.2x2.5mm, symbol Device:Crystal_GND24
- C1, C2, C3, C5, C7: footprint Capacitor_SMD:C_0805_2012Metric -> Capacitor_SMD:C_0805_2012Metric_Pad1.15x1.40mm_HandSolder
- D4, D5: footprint LED_SMD:LED_0805_2012Metric -> LED_SMD:LED_0805_2012Metric_Pad1.15x1.40mm_HandSolder
- P1: renamed from P2; footprint Connector_PinHeader_2.54mm:PinHeader_1x09_P2.54mm_Vertical -> Connector_PinHeader_2.54mm:PinHeader_1x08_P2.54mm_Vertical; symbol Connector_Generic:Conn_01x09 -> Connector_Generic:Conn_01x08
- P2: renamed from P3; footprint Socket_Arduino_Uno:Socket_Strip_Arduino_1x06 -> Connector_PinHeader_2.54mm:PinHeader_1x06_P2.54mm_Vertical
- P4: renamed from P1; footprint Socket_Arduino_Uno:Socket_Strip_Arduino_1x06 -> Connector_PinHeader_2.54mm:PinHeader_1x06_P2.54mm_Vertical
- P6: renamed from P4; footprint Socket_Arduino_Uno:Socket_Strip_Arduino_1x08 -> Connector_PinHeader_2.54mm:PinHeader_1x08_P2.54mm_Vertical
- R1: renamed from R2; footprint Resistor_SMD:R_0805_2012Metric -> Resistor_SMD:R_0805_2012Metric_Pad1.15x1.40mm_HandSolder
- R4: renamed from R6; footprint Resistor_SMD:R_0805_2012Metric -> Resistor_SMD:R_0805_2012Metric_Pad1.15x1.40mm_HandSolder
- R5: footprint Resistor_SMD:R_0805_2012Metric -> Resistor_SMD:R_0805_2012Metric_Pad1.15x1.40mm_HandSolder
- R6: renamed from R7; footprint Resistor_SMD:R_0805_2012Metric -> Resistor_SMD:R_0805_2012Metric_Pad1.15x1.40mm_HandSolder
- U3: footprint (none) -> Package_SO:SOIC-8_3.9x4.9mm_P1.27mm
- renumbered D6 to D7, J4 to J3, J2 to J4
Connections:
- net +5V: now also P1.1 (Pin_1), R2.1, R3.1; no longer P1.4 (Pin_4), R5.1
- net A0: now also P5.1 (Pin_1)
- net A1: now also P5.2 (Pin_2)
- net A2: now also P5.3 (Pin_3)
- net A3: now also P5.4 (Pin_4)
- net A4(SDA): now also P5.5 (Pin_5)
- net A5(SCL): now also P5.6 (Pin_6)
- net AREF: now also P1.8 (Pin_8); no longer P1.9 (Pin_9)
- net GND: now also P1.5 (Pin_5), D6.1 (K), J2.2 (Pin_2), Y1.2, Y1.4; no longer P1.8 (Pin_8)
- net PB0(8): now also P3.1 (Pin_1), U3.5 (+)
- net PB1(9): now also P3.2 (Pin_2)
- net PB2(SS): now also P3.3 (Pin_3)
- net PB3(MOSI): now also P3.4 (Pin_4)
- net PB4(MISO): now also P3.5 (Pin_5)
- net PB5(SCK): now also P3.6 (Pin_6)
- net PD2: now also P7.3 (Pin_3)
- net PD3: now also P7.4 (Pin_4)
- net PD4: now also P7.5 (Pin_5)
- net PD5: now also P7.6 (Pin_6)
- net PD6: now also P7.7 (Pin_7)
- net PD7: now also P7.8 (Pin_8)
- net Reset: now also P1.4 (Pin_4), R7.2; no longer P1.5 (Pin_5), SW1.1
- net Rx: now also D3.1 (K), P7.1 (Pin_1)
- net Tx: now also D2.1 (K), P7.2 (Pin_2)
- net XTAL1: now also Y1.3
- net XTAL2: now also Y1.1
- net at D4.2 (A), R1.2: no longer R5.2
- net Vin: no longer names the net of D1.2 (A), J1.1
- net Vin: now also J2.1 (Pin_1); no longer P1.1 (Pin_1)
- new net: R7.1, SW1.1
- new net: D2.2 (A), R2.2
- new net: D3.2 (A), R3.2
- new net: R5.1, U3.6 (-), U3.7
- new net: D6.2 (A), R5.2
- no-connect marks 1 -> 0
Other:
- moved on the sheet: C7, D5, D7, J3, J4, P2, P4, P6, R4, R6, SW1, U3A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

Commit message: Use proper cap values for crystal
Parts:
- C3, C5: value 22pF -> 30pF
Changed lines of the file:
@@
 P 3950 9650
 F 0 "C5" H 3835 9604 50  0000 R CNN
-F 1 "22pF" H 3835 9695 50  0000 R CNN
+F 1 "30pF" H 3835 9695 50  0000 R CNN
 F 2 "Capacitor_SMD:C_0805_2012Metric_Pad1.15x1.40mm_HandSolder" H 3988 9500 50  0001 C CNN
 F 3 "~" H 3950 9650 50  0001 C CNN
@@
 P 2950 9650
 F 0 "C3" H 2835 9604 50  0000 R CNN
-F 1 "22pF" H 2835 9695 50  0000 R CNN
+F 1 "30pF" H 2835 9695 50  0000 R CNN
 F 2 "Capacitor_SMD:C_0805_2012Metric_Pad1.15x1.40mm_HandSolder" H 2988 9500 50  0001 C CNN
 F 3 "~" H 2950 9650 50  0001 C CNN
